File: TestIC.kicad_sch (KiCad schematic)
At the start: 2 parts, among them U1 74LS02, U2 74LS02

Commit message: WIP - Updated code to work in separate phases:
-Read schematics into classes
-Generate netlists - working!
-Write verilog files (still needs to write pins properly)
Also:
-added verilog library with NOT and NOR2 symbols
-added parsing of each page, even the top one, in case you want a design with a single page
Parts:
- removed U1, U2: 74LS02, symbol 74xx:74LS02
- added U1, U2: NOR2, symbol VerilogLibrary:NOR2
Connections:
- net CLK: now also U1.2, U2.3
- net inv/A: now also U1.1, U2.2
- net inv1/A: now also U1.3, U2.1
Changed lines of the file:
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@@
+    (stroke (width 0) (type default) (color 0 0 0 0))
+  )
+  (wire (pts (xy 100.33 50.8) (xy 107.95 50.8))
     (stroke (width 0) (type default) (color 0 0 0 0))
   )
@@
   )
   (wire (pts (xy 107.95 55.88) (xy 77.47 55.88))
-    (stroke (width 0) (type default) (color 0 0 0 0))
-  )
-  (wire (pts (xy 100.33 50.8) (xy 107.95 50.8))
     (stroke (width 0) (type default) (color 0 0 0 0))
   )
@@
     (effects (font (size 1.27 1.27)) (justify left))
   )
-  (symbol (lib_id "74xx:74LS02") (at 92.71 50.8 0) (unit 1)
+  (symbol (lib_id "VerilogLibrary:NOR2") (at 92.71 69.85 0) (unit 1)
+    (in_bom yes) (on_board yes) (fields_autoplaced)
+    (property "Reference" "U2" (id 0) (at 92.71 60.96 0))
+    (property "Value" "NOR2" (id 1) (at 92.71 63.5 0))
+    (property "Footprint" "" (id 2) (at 92.71 69.85 0)
+      (effects (font (size 1.27 1.27)) hide)
+    )
+    (property "Datasheet" "http://www.ti.com/lit/gpn/sn74ls02" (id 3) (at 92.71 69.85 0)
+      (effects (font (size 1.27 1.27)) hide)
+    )
+    (pin "1")
+    (pin "2")
+    (pin "3")
+  )
+  (symbol (lib_id "VerilogLibrary:NOR2") (at 92.71 50.8 0) (unit 1)
     (in_bom yes) (on_board yes) (fields_autoplaced)
     (property "Reference" "U1" (id 0) (at 92.71 41.91 0))
-    (property "Value" "74LS02" (id 1) (at 92.71 44.45 0))
+    (property "Value" "NOR2" (id 1) (at 92.71 44.45 0))
     (property "Footprint" "" (id 2) (at 92.71 50.8 0)
       (effects (font (size 1.27 1.27)) hide)
@@
       (effects (font (size 1.27 1.27)) hide)
     )
-    (pin "1")
-    (pin "2")
-    (pin "3")
-  )
-  (symbol (lib_id "74xx:74LS02") (at 92.71 69.85 0) (unit 1)
-    (in_bom yes) (on_board yes) (fields_autoplaced)
-    (property "Reference" "U2" (id 0) (at 92.71 60.96 0))
-    (property "Value" "74LS02" (id 1) (at 92.71 63.5 0))
-    (property "Footprint" "" (id 2) (at 92.71 69.85 0)
-      (effects (font (size 1.27 1.27)) hide)
-    )
-    (property "Datasheet" "http://www.ti.com/lit/gpn/sn74ls02" (id 3) (at 92.71 69.85 0)
-      (effects (font (size 1.27 1.27)) hide)
-    )
