File: kicadtoverilog_test/TestIC.kicad_sch (KiCad schematic)
At the start: 2 parts, among them U1 NOR2, U2 NOR2

Commit message: Restructure project - verilog structure should be correct now
Connections:
- net CLK: now also U1.1, U2.2; no longer U1.2, U2.3
- net inv/A: now also U1.3, U2.1; no longer U1.1, U2.2
- net inv1/A: now also U1.2, U2.3; no longer U1.3, U2.1
Changed lines of the file:
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@@
     (effects (font (size 1.27 1.27)) (justify left))
+  )
+  (symbol (lib_id "VerilogLibrary:NOR2") (at 92.71 50.8 0) (unit 1)
+    (in_bom yes) (on_board yes) (fields_autoplaced)
+    (property "Reference" "U1" (id 0) (at 92.71 41.91 0))
+    (property "Value" "NOR2" (id 1) (at 92.71 44.45 0))
+    (property "Footprint" "" (id 2) (at 92.71 50.8 0)
+      (effects (font (size 1.27 1.27)) hide)
+    )
+    (property "Datasheet" "http://www.ti.com/lit/gpn/sn74ls02" (id 3) (at 92.71 50.8 0)
+      (effects (font (size 1.27 1.27)) hide)
+    )
+    (pin "1")
+    (pin "2")
+    (pin "3")
   )
   (symbol (lib_id "VerilogLibrary:NOR2") (at 92.71 69.85 0) (unit 1)
@@
       (effects (font (size 1.27 1.27)) hide)
     )
-    (pin "1")
-    (pin "2")
-    (pin "3")
-  )
-  (symbol (lib_id "VerilogLibrary:NOR2") (at 92.71 50.8 0) (unit 1)
-    (in_bom yes) (on_board yes) (fields_autoplaced)
-    (property "Reference" "U1" (id 0) (at 92.71 41.91 0))
-    (property "Value" "NOR2" (id 1) (at 92.71 44.45 0))
-    (property "Footprint" "" (id 2) (at 92.71 50.8 0)
-      (effects (font (size 1.27 1.27)) hide)
-    )
-    (property "Datasheet" "http://www.ti.com/lit/gpn/sn74ls02" (id 3) (at 92.71 50.8 0)
-      (effects (font (size 1.27 1.27)) hide)
-    )

Commit message: Update symbol pins to use pin names and not pin numbers, to match sheets
Update module/sheet names to drop the '_kicad_sch' suffix
Connections:
- net inv/A is gone; now on net inv1/A: U1.3 (Y), U2.1 (A)
- net inv1/A: no longer U1.2, U2.3
- new net inv2/A: U1.2 (B), U2.3 (Y)
Other:
- removed sheet inv
- added sheet inv2 (inv.kicad_sch)
Changed lines of the file:
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@@
     (effects (font (size 1.27 1.27)) (justify left))
   )
-  (symbol (lib_id "VerilogLibrary:NOR2") (at 92.71 50.8 0) (unit 1)
+  (symbol (lib_name "NOR2_1") (lib_id "VerilogLibrary:NOR2") (at 92.71 50.8 0) (unit 1)
     (in_bom yes) (on_board yes) (fields_autoplaced)
     (property "Reference" "U1" (id 0) (at 92.71 41.91 0))
@@
     (stroke (width 0.1524) (type solid) (color 0 0 0 0))
     (fill (color 0 0 0 0.0000))
-    (property "Sheet name" "inv" (id 0) (at 121.92 46.2784 0)
+    (property "Sheet name" "inv1" (id 0) (at 121.92 46.2784 0)
       (effects (font (size 1.27 1.27)) (justify left bottom))
     )
@@
     (stroke (width 0.1524) (type solid) (color 0 0 0 0))
     (fill (color 0 0 0 0.0000))
-    (property "Sheet name" "inv1" (id 0) (at 121.92 65.3284 0)
+    (property "Sheet name" "inv2" (id 0) (at 121.92 65.3284 0)
       (effects (font (size 1.27 1.27)) (justify left bottom))
     )
